Commit message: Minor modification

File: chapter6_tutorials/robot_description/urdf/robot_gazebo.xacro (robot description, xacro)
@@ -25,5 +25,5 @@
 		<xacro:default_inertial mass="0.0001"/>
  	</link>
- 	<xacro:include filename="$(find robot1_description)/urdf/robot.gazebo" />
+ 	<xacro:include filename="$(find robot_description)/urdf/robot.gazebo" />
 	<gazebo reference="base_footprint">
 		<material>Gazebo/Green</material>
@@ -192,5 +192,5 @@
       <origin xyz="0 0 0" rpy="0 0 0"/>
       <geometry>
-        <mesh filename="package://robot1_description/meshes/hokuyo.dae"/>
+        <mesh filename="package://robot_description/meshes/hokuyo.dae"/>
       </geometry>
     </visual>
